Commit message: removed unused files

File: bender_description/urdf/sensors/_d435.urdf.xacro (robot description, xacro)
@@ -8,5 +8,5 @@
 <robot name="sensor_d435" xmlns:xacro="http://ros.org/wiki/xacro">
   <!--File includes-->
-  <xacro:include filename="$(find magni_description)/urdf/sensors/_d435.gazebo.xacro"/>
+  <xacro:include filename="$(find bender_description)/urdf/sensors/_d435.gazebo.xacro"/>
   <xacro:macro name="sensor_d435" params="name:=camera topics_ns:=camera parent *origin publish_pointcloud:=false">
     <xacro:property name="M_PI" value="3.1415926535897931" />
@@ -49,5 +49,5 @@
         <geometry>
           <!-- <box size="${d435_cam_width} ${d435_cam_height} ${d435_cam_depth}"/> -->
-          <mesh filename="package://magni_description/meshes/sensors/d435.dae" />
+          <mesh filename="package://bender_description/meshes/sensors/d435.dae" />
           <!--<mesh filename="package://realsense2_description/meshes/d435/d435.dae" />-->
         </geometry>

File: bender_description/urdf/sensors/raspi_camera.xacro (robot description, xacro)
@@ -13,5 +13,5 @@
         <origin xyz="0 0 0" rpy="${pi/2} 0 0" />
         <geometry>
-          <mesh filename="package://magni_description/meshes/sensors/raspi_camera.dae" />
+          <mesh filename="package://bender_description/meshes/sensors/raspi_camera.dae" />
         </geometry>
       </visual>

File: bender_description/urdf/sensors/sonar_hc-sr04.xacro (robot description, xacro)
@@ -13,5 +13,5 @@
         <origin xyz="-0.006 0 0" rpy="${pi/2} 0 ${pi/2}" />
         <geometry>
-          <mesh filename="package://magni_description/meshes/sensors/sonar_hc-sr04.dae" />
+          <mesh filename="package://bender_description/meshes/sensors/sonar_hc-sr04.dae" />
         </geometry>
       </visual>
