Commit message: update frames to follow REP-105, 120

File: bender_description/urdf/bender.urdf.xacro (robot description, xacro)
@@ -49,5 +49,5 @@
 	<xacro:include filename="$(find bender_description)/urdf/materials.xacro" />
 	<!-- BODY link -->
-	<link name="body">
+	<link name="base_link">
 		<collision>
 			<origin xyz="0 0 0" rpy="0 0 0"/>
@@ -71,8 +71,14 @@
 		</inertial>
 	</link>
+	<link name="base_footprint"/>
+	<joint name="base_footprint_joint" type="fixed">
+		<parent link="base_footprint"/>
+		<child link="base_link"/>
+		<origin xyz="0 0 ${height + body_h/2}" rpy="0 0 0"/>
+	</joint>
 	<!-- LEG joints -->
 	<joint name="leg_lf_joint" type="continuous">
 		<origin xyz="${body_l / 2} ${body_w / 2} ${-body_h/2 - (height - 2*wheel_r - wheel_off)/2}" rpy="0 0 0"/>
-		<parent link="body" />
+		<parent link="base_link" />
 		<child link="leg_lf" />
 		<dynamics damping="${joint_damping}"/>
@@ -81,5 +87,5 @@
 	<joint name="leg_rf_joint" type="continuous">
 		<origin xyz="${body_l / 2} ${-body_w / 2} ${-body_h/2 - (height - 2*wheel_r - wheel_off)/2}" rpy="0 0 0"/>
-		<parent link="body" />
+		<parent link="base_link" />
 		<child link="leg_rf" />
 		<dynamics damping="${joint_damping}"/>
@@ -88,5 +94,5 @@
 	<joint name="leg_lh_joint" type="continuous">
 		<origin xyz="${-body_l / 2} ${body_w / 2} ${-body_h/2 - (height - 2*wheel_r - wheel_off)/2}" rpy="0 0 0"/>
-		<parent link="body" />
+		<parent link="base_link" />
 		<child link="leg_lh" />
 		<dynamics damping="${joint_damping}"/>
@@ -95,5 +101,5 @@
 	<joint name="leg_rh_joint" type="continuous">
 		<origin xyz="${-body_l / 2} ${-body_w / 2} ${-body_h/2 - (height - 2*wheel_r - wheel_off)/2}" rpy="0 0 0"/>
-		<parent link="body" />
+		<parent link="base_link" />
 		<child link="leg_rh" />
 		<dynamics damping="${joint_damping}"/>

Commit message: urdf, swerve_ctrl, odom w/ correct wheel y-axis

File: bender_description/urdf/bender.urdf.xacro (robot description, xacro)
@@ -206,5 +206,5 @@
 		<parent link="leg_rf"/>
 		<child link="wheel_rf"/>
-		<origin xyz="0 0 ${-(height + wheel_off) / 2}" rpy="0 0 0"/>
+		<origin xyz="0 0 ${-(height + wheel_off) / 2}" rpy="0 0 ${PI}"/>
 		<dynamics damping="${joint_damping}"/>
 		<axis xyz="0 1 0"/>
@@ -220,5 +220,5 @@
 		<parent link="leg_rh"/>
 		<child link="wheel_rh"/>
-		<origin xyz="0 0 ${-(height + wheel_off) / 2}" rpy="0 0 0"/>
+		<origin xyz="0 0 ${-(height + wheel_off) / 2}" rpy="0 0 ${PI}"/>
 		<dynamics damping="${joint_damping}"/>
 		<axis xyz="0 1 0"/>

Commit message: vision stuff simulated w/ gazebo

File: bender_description/urdf/bender.urdf.xacro (robot description, xacro)
@@ -32,4 +32,5 @@
 	<!-- Constants for robot dimensions -->
 	<xacro:property name="PI" value="3.1415926535897931"/>
+	<xacro:property name="DEG2RAD" value="0.017453292519943295"/>
 	<xacro:property name="height" value="0.5" /> <!-- height of the body -->
 	<xacro:property name="body_m" value="25.0" /> <!-- mass of the body structure -->
@@ -44,8 +45,12 @@
 	<xacro:property name="wheel_off" value="0.01" /> <!-- thickness of the wheels -->
 	<xacro:property name="joint_damping" value="1" /> <!-- damping of all joints -->
+	<xacro:property name="camera_mount_height" value="1" />
+	<xacro:property name="camera_tilt_angle_deg" value="15" />
 	<!-- Import all Gazebo-customization elements, including Gazebo colors -->
 	<xacro:include filename="$(find bender_description)/urdf/bender.gazebo" />
 	<!-- Import Rviz colors -->
 	<xacro:include filename="$(find bender_description)/urdf/materials.xacro" />
+	<!-- Import Sensors -->
+	<xacro:include filename="$(find bender_description)/urdf/sensors/logitech_c910.xacro" />
 	<!-- BODY link -->
 	<link name="base_link">
@@ -313,5 +318,9 @@
 		</inertial>
 	</link>
-	<!-- SENSORS: nothing yet -->
+	<!-- SENSORS: -->
+	<xacro:logitech_c910 name="logitech_cam" connected_to="base_link">
+		<origin xyz="${-body_l/2} 0 ${camera_mount_height}"
+			    rpy="0 ${camera_tilt_angle_deg*DEG2RAD} 0" />
+    </xacro:logitech_c910>
 	<!-- ACTUATORS -->
 	<transmission name="leg_lf_trans">

Commit message: added lidar

File: bender_description/urdf/bender.urdf.xacro (robot description, xacro)
@@ -47,4 +47,5 @@
 	<xacro:property name="camera_mount_height" value="1" />
 	<xacro:property name="camera_tilt_angle_deg" value="15" />
+	<xacro:property name="lidar_mount_height" value="0.0" />
 	<!-- Import all Gazebo-customization elements, including Gazebo colors -->
 	<xacro:include filename="$(find bender_description)/urdf/bender.gazebo" />
@@ -53,4 +54,5 @@
 	<!-- Import Sensors -->
 	<xacro:include filename="$(find bender_description)/urdf/sensors/logitech_c910.xacro" />
+	<xacro:include filename="$(find bender_description)/urdf/sensors/rplidar.xacro" />
 	<!-- BODY link -->
 	<link name="base_link">
@@ -320,7 +322,11 @@
 	<!-- SENSORS: -->
 	<xacro:logitech_c910 name="logitech_cam" connected_to="base_link">
-		<origin xyz="${-body_l/2} 0 ${camera_mount_height}"
+		<origin xyz="${-body_l/2} 0 ${body_h/2 + camera_mount_height}"
 			    rpy="0 ${camera_tilt_angle_deg*DEG2RAD} 0" />
     </xacro:logitech_c910>
+	<xacro:rplidar name="rplidar" connected_to="base_link">
+		<origin xyz="${body_l/2} 0 ${body_h/2 + lidar_mount_height}"
+			    rpy="0 0 0" />
+    </xacro:rplidar>
 	<!-- ACTUATORS -->
 	<transmission name="leg_lf_trans">

Commit message: axis orientation

File: bender_description/urdf/bender.urdf.xacro (robot description, xacro)
@@ -41,5 +41,5 @@
 	<xacro:property name="leg_r" value="0.025" /> <!-- radius of the leg cylinders -->
 	<xacro:property name="wheel_m" value="5" /> <!-- mass of a single wheel -->
-	<xacro:property name="wheel_r" value="0.15" /> <!-- radius of the wheels -->
+	<xacro:property name="wheel_r" value="0.1" /> <!-- radius of the wheels -->
 	<xacro:property name="wheel_h" value="0.05" /> <!-- thickness of the wheels -->
 	<xacro:property name="wheel_off" value="0.01" /> <!-- thickness of the wheels -->
@@ -206,5 +206,5 @@
 		<parent link="leg_lf"/>
 		<child link="wheel_lf"/>
-		<origin xyz="0 0 ${-(height + wheel_off) / 2}" rpy="0 0 0"/>
+		<origin xyz="0 0 ${-(height + wheel_off) / 2}" rpy="0 0 ${PI}"/>
 		<dynamics damping="${joint_damping}"/>
 		<axis xyz="0 1 0"/>
@@ -213,5 +213,5 @@
 		<parent link="leg_rf"/>
 		<child link="wheel_rf"/>
-		<origin xyz="0 0 ${-(height + wheel_off) / 2}" rpy="0 0 ${PI}"/>
+		<origin xyz="0 0 ${-(height + wheel_off) / 2}" rpy="0 0 0"/>
 		<dynamics damping="${joint_damping}"/>
 		<axis xyz="0 1 0"/>
@@ -220,5 +220,5 @@
 		<parent link="leg_lh"/>
 		<child link="wheel_lh"/>
-		<origin xyz="0 0 ${-(height + wheel_off) / 2}" rpy="0 0 0"/>
+		<origin xyz="0 0 ${-(height + wheel_off) / 2}" rpy="0 0 ${PI}"/>
 		<dynamics damping="${joint_damping}"/>
 		<axis xyz="0 1 0"/>
@@ -227,5 +227,5 @@
 		<parent link="leg_rh"/>
 		<child link="wheel_rh"/>
-		<origin xyz="0 0 ${-(height + wheel_off) / 2}" rpy="0 0 ${PI}"/>
+		<origin xyz="0 0 ${-(height + wheel_off) / 2}" rpy="0 0 0"/>
 		<dynamics damping="${joint_damping}"/>
 		<axis xyz="0 1 0"/>

Commit message: adjusting nav and sim params

File: bender_description/urdf/bender.urdf.xacro (robot description, xacro)
@@ -41,8 +41,8 @@
 	<xacro:property name="leg_r" value="0.025" /> <!-- radius of the leg cylinders -->
 	<xacro:property name="wheel_m" value="5" /> <!-- mass of a single wheel -->
-	<xacro:property name="wheel_r" value="0.1" /> <!-- radius of the wheels -->
+	<xacro:property name="wheel_r" value="0.11" /> <!-- radius of the wheels -->
 	<xacro:property name="wheel_h" value="0.05" /> <!-- thickness of the wheels -->
 	<xacro:property name="wheel_off" value="0.01" /> <!-- thickness of the wheels -->
-	<xacro:property name="joint_damping" value="1" /> <!-- damping of all joints -->
+	<xacro:property name="joint_damping" value="0.1" /> <!-- damping of all joints -->
 	<xacro:property name="camera_mount_height" value="1" />
 	<xacro:property name="camera_tilt_angle_deg" value="15" />

Commit message: hardware fixes

File: bender_description/urdf/bender.urdf.xacro (robot description, xacro)
@@ -35,11 +35,11 @@
 	<xacro:property name="height" value="0.5" /> <!-- height of the body -->
 	<xacro:property name="body_m" value="25.0" /> <!-- mass of the body structure -->
-	<xacro:property name="body_l" value="1.2" /> <!-- length of the body structure -->
-	<xacro:property name="body_w" value="0.8" /> <!-- width of the body structure -->
+	<xacro:property name="body_l" value="0.673" /> <!-- length of the body structure -->
+	<xacro:property name="body_w" value="0.635" /> <!-- width of the body structure -->
 	<xacro:property name="body_h" value="0.2" /> <!-- thickness of the body structure -->
 	<xacro:property name="leg_m" value="1" /> <!-- mass of a thigh leg -->
 	<xacro:property name="leg_r" value="0.025" /> <!-- radius of the leg cylinders -->
 	<xacro:property name="wheel_m" value="5" /> <!-- mass of a single wheel -->
-	<xacro:property name="wheel_r" value="0.11" /> <!-- radius of the wheels -->
+	<xacro:property name="wheel_r" value="0.102" /> <!-- radius of the wheels -->
 	<xacro:property name="wheel_h" value="0.05" /> <!-- thickness of the wheels -->
 	<xacro:property name="wheel_off" value="0.01" /> <!-- thickness of the wheels -->

Commit message: vision config pipeline done, ready for hardware

File: bender_description/urdf/bender.urdf.xacro (robot description, xacro)
@@ -32,5 +32,4 @@
 	<!-- Constants for robot dimensions -->
 	<xacro:property name="PI" value="3.1415926535897931"/>
-	<xacro:property name="DEG2RAD" value="0.017453292519943295"/>
 	<xacro:property name="height" value="0.5" /> <!-- height of the body -->
 	<xacro:property name="body_m" value="25.0" /> <!-- mass of the body structure -->
@@ -321,7 +320,7 @@
 	</link>
 	<!-- SENSORS: -->
-	<xacro:logitech_c910 name="bender_camera" connected_to="base_link">
+	<xacro:logitech_c910 name="bender_camera" connected_to="base_link" tilt_degrees="${camera_tilt_angle_deg}">
 		<origin xyz="${-body_l/2} 0 ${body_h/2 + camera_mount_height}"
-			    rpy="0 ${camera_tilt_angle_deg*DEG2RAD} 0" />
+			    rpy="0 0 0" />
     </xacro:logitech_c910>
 	<xacro:rplidar name="rplidar" connected_to="base_link">

File: bender_description/urdf/sensors/logitech_c910.xacro (robot description, xacro)
@@ -1,5 +1,6 @@
 <?xml version="1.0" encoding="utf-8"?>
 <robot xmlns:xacro="http://wiki.ros.org/xacro">
-  <xacro:macro name="logitech_c910" params="name:='' connected_to:='' *origin">
+  <xacro:macro name="logitech_c910" params="name:='' connected_to:='' tilt_degrees:='0' *origin">
+  <xacro:property name="DEG2RAD" value="0.017453292519943295"/>
     <xacro:unless value="${connected_to == ''}">
       <joint name="${name}_joint" type="fixed">
@@ -28,5 +29,5 @@
       <parent link="${name}"/>
       <child link="${name}_sensor"/>
-      <origin xyz="0.005 0 0" rpy="0 0 0" />
+      <origin xyz="0.005 0 0" rpy="0 ${tilt_degrees*DEG2RAD} 0" />
     </joint>
     <!-- Gazebo sensor plugin -->
@@ -43,5 +44,5 @@
           </image>
           <clip>
-            <near>0.02</near>
+            <near>0.03</near>
             <far>300</far>
           </clip>

Commit message: parameter to adjust laser distance scale

File: bender_description/urdf/bender.urdf.xacro (robot description, xacro)
@@ -32,9 +32,9 @@
 	<!-- Constants for robot dimensions -->
 	<xacro:property name="PI" value="3.1415926535897931"/>
-	<xacro:property name="height" value="0.5" /> <!-- height of the body -->
+	<xacro:property name="height" value="0.3" /> <!-- height of the body -->
 	<xacro:property name="body_m" value="25.0" /> <!-- mass of the body structure -->
 	<xacro:property name="body_l" value="0.673" /> <!-- length of the body structure -->
 	<xacro:property name="body_w" value="0.635" /> <!-- width of the body structure -->
-	<xacro:property name="body_h" value="0.2" /> <!-- thickness of the body structure -->
+	<xacro:property name="body_h" value="0.105" /> <!-- thickness of the body structure -->
 	<xacro:property name="leg_m" value="1" /> <!-- mass of a thigh leg -->
 	<xacro:property name="leg_r" value="0.025" /> <!-- radius of the leg cylinders -->
@@ -44,5 +44,5 @@
 	<xacro:property name="wheel_off" value="0.01" /> <!-- thickness of the wheels -->
 	<xacro:property name="joint_damping" value="0.1" /> <!-- damping of all joints -->
-	<xacro:property name="camera_mount_height" value="1" />
+	<xacro:property name="camera_mount_height" value="0.94" />
 	<xacro:property name="camera_tilt_angle_deg" value="15" />
 	<xacro:property name="lidar_mount_height" value="0.0" />

Commit message: bender3.0 dimensions in urdf

File: bender_description/urdf/bender.urdf.xacro (robot description, xacro)
@@ -34,13 +34,13 @@
 	<xacro:property name="height" value="0.3" /> <!-- height of the body -->
 	<xacro:property name="body_m" value="25.0" /> <!-- mass of the body structure -->
-	<xacro:property name="body_l" value="0.673" /> <!-- length of the body structure -->
-	<xacro:property name="body_w" value="0.635" /> <!-- width of the body structure -->
+	<xacro:property name="body_l" value="0.857" /> <!-- length of the body structure -->
+	<xacro:property name="body_w" value="0.622" /> <!-- width of the body structure -->
 	<xacro:property name="body_h" value="0.105" /> <!-- thickness of the body structure -->
 	<xacro:property name="leg_m" value="1" /> <!-- mass of a thigh leg -->
 	<xacro:property name="leg_r" value="0.025" /> <!-- radius of the leg cylinders -->
 	<xacro:property name="wheel_m" value="5" /> <!-- mass of a single wheel -->
-	<xacro:property name="wheel_r" value="0.102" /> <!-- radius of the wheels -->
+	<xacro:property name="wheel_r" value="0.127" /> <!-- radius of the wheels -->
 	<xacro:property name="wheel_h" value="0.05" /> <!-- thickness of the wheels -->
-	<xacro:property name="wheel_off" value="0.01" /> <!-- thickness of the wheels -->
+	<xacro:property name="wheel_off" value="0.00" /> <!-- thickness of the wheels -->
 	<xacro:property name="joint_damping" value="0.1" /> <!-- damping of all joints -->
 	<xacro:property name="camera_mount_height" value="0.94" />

Commit message: the night before

File: bender_description/urdf/bender.urdf.xacro (robot description, xacro)
@@ -32,9 +32,9 @@
 	<!-- Constants for robot dimensions -->
 	<xacro:property name="PI" value="3.1415926535897931"/>
-	<xacro:property name="height" value="0.3" /> <!-- height of the body -->
+	<xacro:property name="height" value="0.33" /> <!-- height of the body -->
 	<xacro:property name="body_m" value="25.0" /> <!-- mass of the body structure -->
-	<xacro:property name="body_l" value="0.857" /> <!-- length of the body structure -->
+	<xacro:property name="body_l" value="0.904" /> <!-- length of the body structure -->
 	<xacro:property name="body_w" value="0.622" /> <!-- width of the body structure -->
-	<xacro:property name="body_h" value="0.105" /> <!-- thickness of the body structure -->
+	<xacro:property name="body_h" value="0.4191" /> <!-- thickness of the body structure -->
 	<xacro:property name="leg_m" value="1" /> <!-- mass of a thigh leg -->
 	<xacro:property name="leg_r" value="0.025" /> <!-- radius of the leg cylinders -->
@@ -326,5 +326,5 @@
 	<xacro:rplidar name="rplidar" connected_to="base_link">
 		<origin xyz="${body_l/2} 0 ${body_h/2 + lidar_mount_height}"
-			    rpy="0 0 0" />
+			    rpy="0 0 ${PI}" />
     </xacro:rplidar>
 	<!-- ACTUATORS -->
